File: RobotPCB/RobotPowerSupply/RobotPowerSupply.kicad_pcb (KiCad board)
At the start: 2 copper layers, 23 parts, among them J1 Battery, J10 Servo, J11 USB_A_Stacked, J12 USB_A_Stacked, J13 Charging, J14 Charging, J15 MotorL, J16 Servo, J17 Servo, J18 LMotor_Bat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

Commit message: Changing Board a little
Parts:
- moved J3 37.9 mm to (119.7, 76.2), turned to 90 degrees
- moved SW1 33.1 mm to (111.7, 81.6), turned to 0 degrees
Connections:
- J10 pad 3: GND -> -12V
- J11 pad 4: GND -> -12V
- J11 pad 8: GND -> -12V
- J11 pad 9: GND -> -12V
- J12 pad 4: GND -> -12V
- J12 pad 8: GND -> -12V
- J12 pad 9: GND -> -12V
- J15 pad 1: GND -> -12V
- J16 pad 3: GND -> -12V
- J17 pad 3: GND -> -12V
- J18 pad 1: GND -> -12V
- J2 pad 2: GND -> -12V
- J2 pad 3: GND -> -12V
- J3 pad 2: GND -> -12V
- J3 pad 3: GND -> -12V
- J4 pad 2: GND -> -12V
- J5 pad 2: GND -> -12V
- J6 pad 1: GND -> -12V
- J8 pad 1: GND -> -12V
- J9 pad 3: GND -> -12V
- SW1 pad 2: -12V -> OUT1
Routing:
- net -12V: track 0.00 -> 41.3 mm
- net +12V: track 94.6 -> 124.5 mm
- net OUT1: track 0.00 -> 25.1 mm
- net Net-(D2-Pad2): track 161.5 -> 137.4 mm
