File: RobotPCB/RobotPowerSupply/RobotPowerSupply.kicad_sch (KiCad schematic)
At the start: 23 parts, among them J1 Battery, J10 Servo, J11 USB_A_Stacked, J12 USB_A_Stacked, J13 Charging, J14 Charging, J15 MotorL, J16 Servo, J17 Servo, J18 LMotor_Bat, J2 VOut, J3 Output, J4 Hohlstecker, J5 Hohlstecker, J6 RMotor_Bat, J7 Solar, J8 MotorR, J9 Servo, SW1 ON_OFF

Commit message: Changing Board a little
Connections:
- net -12V: now also J10.3 (Pin_3), J11.4 (GND1), J11.8 (GND2), J11.9 (Shield), J12.4 (GND1), J12.8 (GND2), J12.9 (Shield), J15.1 (Pin_1), J16.3 (Pin_3), J17.3 (Pin_3), J18.1 (Pin_1), J2.2 (Pin_2), J2.3 (Pin_3), J3.2 (Pin_2), J3.3 (Pin_3), J4.2, J5.2, J6.1 (Pin_1), J8.1 (Pin_1), J9.3 (Pin_3); no longer SW1.2
- removed net GND: J10.3 (Pin_3), J11.4 (GND1), J11.8 (GND2), J11.9 (Shield), J12.4 (GND1), J12.8 (GND2), J12.9 (Shield), J15.1 (Pin_1), J16.3 (Pin_3), J17.3 (Pin_3), J18.1 (Pin_1), J2.2 (Pin_2), J2.3 (Pin_3), J3.2 (Pin_2), J3.3 (Pin_3), J4.2, J5.2, J6.1 (Pin_1), J8.1 (Pin_1), J9.3 (Pin_3), SW1.3
Changed lines of the file:
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@@
   (junction (at 49.53 20.32) (diameter 0) (color 0 0 0 0)
   )
+  (junction (at 36.83 40.64) (diameter 0) (color 0 0 0 0)
+  )
+  (junction (at 215.265 28.575) (diameter 0) (color 0 0 0 0)
+  )
+  (junction (at 36.83 21.59) (diameter 0) (color 0 0 0 0)
+  )
+  (junction (at 21.59 21.59) (diameter 0) (color 0 0 0 0)
+  )
+  (junction (at 259.08 15.875) (diameter 0) (color 0 0 0 0)
+  )
+  (junction (at 26.67 36.83) (diameter 0) (color 0 0 0 0)
+  )
+  (junction (at 21.59 16.51) (diameter 0) (color 0 0 0 0)
+  )
+  (junction (at 21.59 30.48) (diameter 0) (color 0 0 0 0)
+  )
+  (junction (at 36.83 31.75) (diameter 0) (color 0 0 0 0)
+  )
   (junction (at 40.64 22.86) (diameter 0) (color 0 0 0 0)
   )
-  (junction (at 31.75 36.83) (diameter 0) (color 0 0 0 0)
-  )
-  (junction (at 36.83 40.64) (diameter 0) (color 0 0 0 0)
-  )
-  (junction (at 215.265 28.575) (diameter 0) (color 0 0 0 0)
-  )
-  (junction (at 36.83 21.59) (diameter 0) (color 0 0 0 0)
-  )
-  (junction (at 21.59 21.59) (diameter 0) (color 0 0 0 0)
-  )
-  (junction (at 259.08 15.875) (diameter 0) (color 0 0 0 0)
-  )
-  (junction (at 26.67 36.83) (diameter 0) (color 0 0 0 0)
-  )
-  (junction (at 21.59 16.51) (diameter 0) (color 0 0 0 0)
-  )
-  (junction (at 21.59 30.48) (diameter 0) (color 0 0 0 0)
-  )
-  (junction (at 36.83 31.75) (diameter 0) (color 0 0 0 0)
-  )
   (junction (at 29.21 40.64) (diameter 0) (color 0 0 0 0)
   )
@@
     (stroke (width 0) (type default) (color 0 0 0 0))
   )
-  (wire (pts (xy 54.61 36.83) (xy 53.34 36.83))
-    (stroke (width 0) (type default) (color 0 0 0 0))
-  )
   (wire (pts (xy 29.21 40.64) (xy 29.21 41.91))
     (stroke (width 0) (type default) (color 0 0 0 0))
@@
     (stroke (width 0) (type default) (color 0 0 0 0))
   )
+  (wire (pts (xy 39.37 20.32) (xy 39.37 25.4))
+    (stroke (width 0) (type default) (color 0 0 0 0))
+  )
   (wire (pts (xy 262.255 53.34) (xy 259.08 53.34))
     (stroke (width 0) (type default) (color 0 0 0 0))
@@
     (stroke (width 0) (type default) (color 0 0 0 0))
   )
-  (wire (pts (xy 39.37 27.94) (xy 54.61 27.94))
-    (stroke (width 0) (type default) (color 0 0 0 0))
-  )
   (wire (pts (xy 28.575 19.05) (xy 28.575 26.035))
     (stroke (width 0) (type default) (color 0 0 0 0))
   )
+  (wire (pts (xy 30.48 25.4) (xy 30.48 30.48))
+    (stroke (width 0) (type default) (color 0 0 0 0))
+  )
   (wire (pts (xy 234.95 24.13) (xy 234.95 28.575))
     (stroke (width 0) (type default) (color 0 0 0 0))
@@
     (stroke (width 0) (type default) (color 0 0 0 0))
   )
-  (wire (pts (xy 39.37 27.94) (xy 39.37 20.32))
-    (stroke (width 0) (type default) (color 0 0 0 0))
-  )
   (wire (pts (xy 215.265 28.575) (xy 215.265 31.115))
     (stroke (width 0) (type default) (color 0 0 0 0))
@@
     (stroke (width 0) (type default) (color 0 0 0 0))
   )
+  (wire (pts (xy 30.48 30.48) (xy 21.59 30.48))
+    (stroke (width 0) (type default) (color 0 0 0 0))
+  )
   (wire (pts (xy 259.08 53.34) (xy 259.08 15.875))
     (stroke (width 0) (type default) (color 0 0 0 0))
@@
     (stroke (width 0) (type default) (color 0 0 0 0))
   )
+  (wire (pts (xy 38.1 29.21) (xy 38.1 22.86))
+    (stroke (width 0) (type default) (color 0 0 0 0))
+  )
+  (wire (pts (xy 21.59 21.59) (xy 29.21 21.59))
+    (stroke (width 0) (type default) (color 0 0 0 0))
+  )
   (wire (pts (xy 38.1 22.86) (xy 40.64 22.86))
     (stroke (width 0) (type default) (color 0 0 0 0))
   )
-  (wire (pts (xy 40.64 20.32) (xy 39.37 20.32))
-    (stroke (width 0) (type default) (color 0 0 0 0))
-  )
-  (wire (pts (xy 38.1 29.21) (xy 38.1 22.86))
-    (stroke (width 0) (type default) (color 0 0 0 0))
-  )
-  (wire (pts (xy 21.59 21.59) (xy 29.21 21.59))
+  (wire (pts (xy 36.83 40.64) (xy 36.83 41.91))
+    (stroke (width 0) (type default) (color 0 0 0 0))
+  )
+  (wire (pts (xy 207.01 14.605) (xy 213.36 14.605))
+    (stroke (width 0) (type default) (color 0 0 0 0))
+  )
+  (wire (pts (xy 26.67 36.83) (xy 31.75 36.83))
+    (stroke (width 0) (type default) (color 0 0 0 0))
+  )
+  (wire (pts (xy 250.825 48.26) (xy 251.46 48.26))
+    (stroke (width 0) (type default) (color 0 0 0 0))
+  )
+  (wire (pts (xy 38.1 29.21) (xy 53.34 29.21))
+    (stroke (width 0) (type default) (color 0 0 0 0))
+  )
+  (wire (pts (xy 259.08 15.875) (xy 236.22 15.875))
+    (stroke (width 0) (type default) (color 0 0 0 0))
+  )
+  (wire (pts (xy 243.205 36.195) (xy 243.205 28.575))
+    (stroke (width 0) (type default) (color 0 0 0 0))
+  )
+  (wire (pts (xy 253.365 45.72) (xy 253.365 50.165))
+    (stroke (width 0) (type default) (color 0 0 0 0))
+  )
+  (wire (pts (xy 242.57 27.305) (xy 243.205 27.305))
+    (stroke (width 0) (type default) (color 0 0 0 0))
+  )
+  (wire (pts (xy 261.62 31.115) (xy 274.32 31.115))
+    (stroke (width 0) (type default) (color 0 0 0 0))
+  )
+  (wire (pts (xy 257.81 24.765) (xy 257.81 20.955))
+    (stroke (width 0) (type default) (color 0 0 0 0))
+  )
+  (wire (pts (xy 250.825 36.195) (xy 251.46 36.195))
+    (stroke (width 0) (type default) (color 0 0 0 0))
+  )
+  (wire (pts (xy 242.57 33.655) (xy 242.57 27.305))
+    (stroke (width 0) (type default) (color 0 0 0 0))
+  )
+  (wire (pts (xy 262.255 15.875) (xy 259.08 15.875))
+    (stroke (width 0) (type default) (color 0 0 0 0))
+  )
+  (wire (pts (xy 40.64 15.24) (xy 38.1 15.24))
+    (stroke (width 0) (type default) (color 0 0 0 0))
+  )
+  (wire (pts (xy 26.67 36.83) (xy 26.67 45.72))
     (stroke (width 0) (type default) (color 0 0 0 0))
   )
@@
     (stroke (width 0) (type default) (color 0 0 0 0))
   )
-  (wire (pts (xy 36.83 40.64) (xy 36.83 41.91))
-    (stroke (width 0) (type default) (color 0 0 0 0))
-  )
-  (wire (pts (xy 207.01 14.605) (xy 213.36 14.605))
-    (stroke (width 0) (type default) (color 0 0 0 0))
-  )
-  (wire (pts (xy 26.67 36.83) (xy 31.75 36.83))
-    (stroke (width 0) (type default) (color 0 0 0 0))
-  )
-  (wire (pts (xy 250.825 48.26) (xy 251.46 48.26))
-    (stroke (width 0) (type default) (color 0 0 0 0))
-  )
-  (wire (pts (xy 38.1 29.21) (xy 53.34 29.21))
-    (stroke (width 0) (type default) (color 0 0 0 0))
-  )
-  (wire (pts (xy 259.08 15.875) (xy 236.22 15.875))
-    (stroke (width 0) (type default) (color 0 0 0 0))
-  )
-  (wire (pts (xy 243.205 36.195) (xy 243.205 28.575))
-    (stroke (width 0) (type default) (color 0 0 0 0))
-  )
-  (wire (pts (xy 253.365 45.72) (xy 253.365 50.165))
-    (stroke (width 0) (type default) (color 0 0 0 0))
-  )
-  (wire (pts (xy 242.57 27.305) (xy 243.205 27.305))
-    (stroke (width 0) (type default) (color 0 0 0 0))
-  )
-  (wire (pts (xy 261.62 31.115) (xy 274.32 31.115))
-    (stroke (width 0) (type default) (color 0 0 0 0))
-  )
-  (wire (pts (xy 257.81 24.765) (xy 257.81 20.955))
-    (stroke (width 0) (type default) (color 0 0 0 0))
-  )
-  (wire (pts (xy 250.825 36.195) (xy 251.46 36.195))
-    (stroke (width 0) (type default) (color 0 0 0 0))
-  )
-  (wire (pts (xy 242.57 33.655) (xy 242.57 27.305))
-    (stroke (width 0) (type default) (color 0 0 0 0))
-  )
-  (wire (pts (xy 262.255 15.875) (xy 259.08 15.875))
-    (stroke (width 0) (type default) (color 0 0 0 0))
-  )
-  (wire (pts (xy 40.64 15.24) (xy 38.1 15.24))
-    (stroke (width 0) (type default) (color 0 0 0 0))
-  )
-  (wire (pts (xy 26.67 36.83) (xy 26.67 45.72))
-    (stroke (width 0) (type default) (color 0 0 0 0))
-  )
   (wire (pts (xy 221.615 15.875) (xy 213.36 15.875))
     (stroke (width 0) (type default) (color 0 0 0 0))
@@
     (stroke (width 0) (type default) (color 0 0 0 0))
   )
+  (wire (pts (xy 39.37 20.32) (xy 40.64 20.32))
+    (stroke (width 0) (type default) (color 0 0 0 0))
+  )
   (wire (pts (xy 261.62 44.45) (xy 274.32 44.45))
     (stroke (width 0) (type default) (color 0 0 0 0))
@@
     (stroke (width 0) (type default) (color 0 0 0 0))
   )
+  (wire (pts (xy 39.37 25.4) (xy 30.48 25.4))
+    (stroke (width 0) (type default) (color 0 0 0 0))
+  )
   (wire (pts (xy 38.1 15.24) (xy 38.1 22.86))
     (stroke (width 0) (type default) (color 0 0 0 0))
@@
     (stroke (width 0) (type default) (color 0 0 0 0))
   )
-  (wire (pts (xy 54.61 27.94) (xy 54.61 36.83))
-    (stroke (width 0) (type default) (color 0 0 0 0))
-  )
   (wire (pts (xy 253.365 50.165) (xy 255.27 50.165))
     (stroke (width 0) (type default) (color 0 0 0 0))
@@
     (stroke (width 0) (type default) (color 0 0 0 0))
   )
-  (wire (pts (xy 31.75 36.83) (xy 38.1 36.83))
-    (stroke (width 0) (type default) (color 0 0 0 0))
-  )
